Commit message: Update drone.urdf.xacro

File: workspace/src/my_robot_description/drone.urdf.xacro (robot description, xacro)
@@ -34,4 +34,51 @@
   </sensor>
 </gazebo>
+<gazebo reference="lidar_link">
+  <sensor name="lidar_sensor" type="ray">
+    <pose>0 0 0 0 0 0</pose>
+    <visualize>true</visualize>
+    <update_rate>10</update_rate>
+    <ray>
+      <scan>
+        <horizontal>
+          <samples>360</samples>
+          <resolution>1</resolution>
+          <min_angle>-3.14</min_angle>
+          <max_angle>3.14</max_angle>
+        </horizontal>
+      </scan>
+      <range>
+        <min>0.1</min>
+        <max>10.0</max>
+        <resolution>0.01</resolution>
+      </range>
+      <noise>
+        <type>gaussian</type>
+        <mean>0.0</mean>
+        <stddev>0.01</stddev>
+      </noise>
+    </ray>
+    <plugin name="gazebo_ros_laser_controller" filename="libgazebo_ros_ray_sensor.so">
+      <ros>
+        <namespace>/</namespace>
+        <remapping>LIDAR_SCAN:=scan</remapping>
+      </ros>
+      <frame_name>lidar_link</frame_name>
+    </plugin>
+  </sensor>
+</gazebo>
+<gazebo reference="barometer_link">
+  <sensor name="baro_sensor" type="altimeter">
+    <pose>0 0 0 0 0 0</pose>
+    <update_rate>10</update_rate>
+    <plugin name="baro_plugin" filename="libgazebo_ros_altimeter.so">
+      <ros>
+        <namespace>/</namespace>
+        <remapping>barometer:=barometer_data</remapping>
+      </ros>
+      <frame_name>barometer_link</frame_name>
+    </plugin>
+  </sensor>
+</gazebo>
 <!--properties-->
     <xacro:property name="arm_length" value="0.225"/>
@@ -175,4 +222,40 @@
         </collision>
     </link>
+    <link name="lidar_link">
+        <visual>
+            <geometry>
+                <cylinder radius="0.03" length="0.02"/>
+            </geometry>
+            <origin xyz="0 0 0" rpy="0 0 0"/>
+            <material name="green"/>
+        </visual>
+        <collision>
+            <geometry>
+                <cylinder radius="0.03" length="0.02"/>
+            </geometry>
+        </collision>
+        <inertial>
+            <mass value="0.2"/>
+            <inertia ixx="1e-5" ixy="0" ixz="0" iyy="1e-5" iyz="0" izz="1e-5"/>
+        </inertial>
+    </link>
+    <link name="barometer_link">
+        <visual>
+            <geometry>
+                <box size="0.02 0.02 0.005"/>
+            </geometry>
+            <origin xyz="0 0 0" rpy="0 0 0"/>
+            <material name="blue"/>
+        </visual>
+        <collision>
+            <geometry>
+                <box size="0.02 0.02 0.005"/>
+            </geometry>
+        </collision>
+        <inertial>
+            <mass value="0.05"/>
+            <inertia ixx="1e-5" ixy="0" ixz="0" iyy="1e-5" iyz="0" izz="1e-5"/>
+        </inertial>
+    </link>
 <!--sensor joints-->
     <joint name="base_imu_joint" type="fixed">
@@ -181,4 +264,14 @@
         <origin xyz="0 0 0" rpy="0 0 0"/>
     </joint>
+    <joint name="lidar_joint" type="fixed">
+        <parent link="base_link"/>
+        <child link="lidar_link"/>
+        <origin xyz="0 0 0.1" rpy="0 0 0"/>
+    </joint>
+    <joint name="barometer_joint" type="fixed">
+        <parent link="base_link"/>
+        <child link="barometer_link"/>
+        <origin xyz="0 0 0.05" rpy="0 0 0"/>
+    </joint>
 <!--sensors-->
 </robot>

Commit message: Update drone.urdf.xacro

File: workspace/src/my_robot_description/drone.urdf.xacro (robot description, xacro)
@@ -1,4 +1,5 @@
 <?xml version="1.0"?>
 <robot xmlns:xacro="http://ros.org/wiki/xacro" name="Udaan">
+<!-- ===== IMU Sensor Plugin Block ===== -->
 <gazebo reference="imu_link">
   <sensor type="imu" name="imu_sensor">
@@ -26,12 +27,13 @@
    <plugin name="imu_plugin" filename="libgazebo_ros_imu_sensor.so">
   <ros>
-    <namespace>imu_plugin</namespace>
     <remapping>imu/data:=/imu/data</remapping>
   </ros>
   <topicName>/imu/data</topicName>
   <frameName>imu_link</frameName>
+  <pose>0 0 0 0 0 0</pose>
    </plugin>
   </sensor>
 </gazebo>
+<!-- ===== LIDAR Sensor Plugin Block ===== -->
 <gazebo reference="lidar_link">
   <sensor name="lidar_sensor" type="ray">
@@ -61,11 +63,12 @@
     <plugin name="gazebo_ros_laser_controller" filename="libgazebo_ros_ray_sensor.so">
       <ros>
-        <namespace>/</namespace>
-        <remapping>LIDAR_SCAN:=scan</remapping>
+        <remapping>LIDAR_SCAN:=/scan</remapping>
       </ros>
       <frame_name>lidar_link</frame_name>
+      <pose>0 0 0 0 0 0</pose>
     </plugin>
   </sensor>
 </gazebo>
+<!-- ===== Barometer Sensor Plugin Block ===== -->
 <gazebo reference="barometer_link">
   <sensor name="baro_sensor" type="altimeter">
@@ -74,8 +77,8 @@
     <plugin name="baro_plugin" filename="libgazebo_ros_altimeter.so">
       <ros>
-        <namespace>/</namespace>
-        <remapping>barometer:=barometer_data</remapping>
+        <remapping>barometer:=/barometer</remapping>
       </ros>
       <frame_name>barometer_link</frame_name>
+      <pose>0 0 0 0 0 0</pose>
     </plugin>
   </sensor>
@@ -112,4 +115,5 @@
             <inertial>
                 <mass value="0.1"/>
+                <origin xyz="0 0 0" rpy="0 0 0"/>
                 <inertia ixx="3.42e-05" ixy="0.0" ixz="0.0"
                          iyy="4.43e-04" iyz="0.0" izz="4.35e-04"/>
@@ -133,4 +137,5 @@
             <inertial>
                 <mass value="0.05"/>
+                 <origin xyz="0 0 0" rpy="0 0 0"/>
                 <inertia ixx="1.32e-05" ixy="0.0" ixz="0.0"
                          iyy="1.32e-05" iyz="0.0" izz="5.63e-06"/>
@@ -169,4 +174,5 @@
         <inertial>
             <mass value="0.750" />
+            <origin xyz="0 0 0" rpy="0 0 0"/>
             <inertia ixx="0.0028125" ixy="0.0" ixz="0.0"
                      iyy="0.0028125" iyz="0.0" izz="0.0015625"/>
@@ -181,7 +187,9 @@
         <material>Gazebo/Red</material>
     </gazebo>
+	<!-- Quad Arm and Motor Placement -->
 <!--top right part-->
     <xacro:arm_link name="top_right_arm" xyz="0.075 0.075 0" rpy="0 0 0.785"/>
     <xacro:motor_link name="motor_top_right_arm" xyz="0 0 0" rpy="0 0 0"/>
+    <!-- Joints: base_link ↔ top_right_arm ↔ motor_top_right_arm -->
     <xacro:fixed_joint name="base_top_right_arm_joint" parent="base_link" child="top_right_arm" xyz="0.065 0.065 0" rpy="0 0 0"/>
     <xacro:motor_joint name="top_right_arm_motor_joint" parent="top_right_arm" child="motor_top_right_arm" xyz="0.125 0.125 0" axis="0 0 -1"/>
@@ -189,4 +197,5 @@
     <xacro:arm_link name="top_left_arm" xyz="-0.075 0.075 0" rpy="0 0 -0.785"/>
     <xacro:motor_link name="motor_top_left_arm" xyz="0 0 0" rpy="0 0 0"/>
+    <!-- Joints: base_link ↔ top_left_arm ↔ motor_top_left_arm -->
     <xacro:fixed_joint name="base_top_left_arm_joint" parent="base_link" child="top_left_arm" xyz="-0.065 0.065 0" rpy="0 0 0"/>
     <xacro:motor_joint name="top_left_arm_motor_joint" parent="top_left_arm" child="motor_top_left_arm" xyz="-0.125 0.125 0" axis="0 0 1"/>
@@ -194,12 +203,15 @@
     <xacro:arm_link name="bottom_right_arm" xyz="0.075 -0.075 0" rpy="0 0 -0.785"/>
     <xacro:motor_link name="motor_bottom_right_arm" xyz="0 0 0" rpy="0 0 0"/>
+    <!-- Joints: base_link ↔ bottom_right_arm ↔ motor_bottom_right_arm -->
     <xacro:fixed_joint name="base_bottom_right_arm_joint" parent="base_link" child="bottom_right_arm" xyz="0.065 -0.065 0" rpy="0 0 0"/>
     <xacro:motor_joint name="bottom_right_arm_motor_joint" parent="bottom_right_arm" child="motor_bottom_right_arm" xyz="0.125 -0.125 0" axis="0 0 1"/>
-<!--bottom left parts-->
+<!--bottom left part-->
     <xacro:arm_link name="bottom_left_arm" xyz="-0.075 -0.075 0" rpy="0 0 -2.35"/>
     <xacro:motor_link name="motor_bottom_left_arm" xyz="0 0 0" rpy="0 0 0"/>
+    <!-- Joints: base_link ↔ bottom_left_arm ↔ motor_bottom_left_arm -->
     <xacro:fixed_joint name="base_bottom_left_arm_joint" parent="base_link" child="bottom_left_arm" xyz="-0.065 -0.065 0" rpy="0 0 0"/>
     <xacro:motor_joint name="bottom_left_arm_motor_joint" parent="bottom_left_arm" child="motor_bottom_left_arm" xyz="-0.125 -0.125 0" axis="0 0 -1"/>
 <!--sensor links-->
+<!-- IMU Sensor Link -->
     <link name="imu_link">
         <visual>
@@ -222,4 +234,5 @@
         </collision>
     </link>
+	<!-- LiDAR Sensor Link -->
     <link name="lidar_link">
         <visual>
@@ -237,7 +250,9 @@
         <inertial>
             <mass value="0.2"/>
+            <origin xyz="0 0 0" rpy="0 0 0"/>
             <inertia ixx="1e-5" ixy="0" ixz="0" iyy="1e-5" iyz="0" izz="1e-5"/>
         </inertial>
     </link>
+<!-- Barometer Sensor Link -->
     <link name="barometer_link">
         <visual>
@@ -255,4 +270,5 @@
         <inertial>
             <mass value="0.05"/>
+            <origin xyz="0 0 0" rpy="0 0 0"/>
             <inertia ixx="1e-5" ixy="0" ixz="0" iyy="1e-5" iyz="0" izz="1e-5"/>
         </inertial>
@@ -276,2 +292,3 @@
 <!--sensors-->
 </robot>
+<!-- END OF ROBOT DEFINITION -->

Commit message: Update drone.urdf.xacro

File: workspace/src/my_robot_description/drone.urdf.xacro (robot description, xacro)
@@ -76,9 +76,6 @@
     <update_rate>10</update_rate>
     <plugin name="baro_plugin" filename="libgazebo_ros_altimeter.so">
-      <ros>
-        <remapping>barometer:=/barometer</remapping>
-      </ros>
+      <topic_name>/barometer/data</topic_name>
       <frame_name>barometer_link</frame_name>
-      <pose>0 0 0 0 0 0</pose>
     </plugin>
   </sensor>
@@ -283,10 +280,10 @@
         <parent link="base_link"/>
         <child link="lidar_link"/>
-        <origin xyz="0 0 0.1" rpy="0 0 0"/>
+        <origin xyz="0 0 0.2" rpy="0 0 0"/>
     </joint>
     <joint name="barometer_joint" type="fixed">
         <parent link="base_link"/>
         <child link="barometer_link"/>
-        <origin xyz="0 0 0.05" rpy="0 0 0"/>
+        <origin xyz="0 0 0.25" rpy="0 0 0"/>
     </joint>
 <!--sensors-->
